File: keyfob.kicad_pcb (KiCad board)
At the start: 2 copper layers, 0 parts

Commit message: PCB layout done
Parts:
- added BZ1: BUZZER, Buzzer_Beeper:Buzzer_15x7.5RM7.6, F.Cu at (123.5, 104.1)
- added C1: 4.7uf, Capacitor_SMD:C_Elec_3x5.4, F.Cu at (136.5, 80.6)
- added C2: 0.1uf, Capacitor_SMD:C_Elec_3x5.4, F.Cu at (137.1, 87.0)
- added D1: LED_KRGB, LED_SMD:LED_RGB_1210, F.Cu at (133.3, 93.4)
- added D2: 3.6V, Diode_SMD:D_0805_2012Metric, F.Cu at (118.9, 78.0)
- added D3: 3.6V, Diode_SMD:D_0805_2012Metric, F.Cu at (116.6, 83.0)
- added D4: D_Schottky, Diode_SMD:D_0805_2012Metric, F.Cu at (121.0, 83.7)
- added H1: MountingHole, MountingHole:MountingHole_4mm, F.Cu at (127.7, 78.5)
- added J2: USB_A, Connector_USB:USB_A_Molex_67643_Horizontal, F.Cu at (124.5, 115.7)
- added PWR1: LED, LED_SMD:LED_0805_2012Metric, F.Cu at (116.7, 88.4)
- added R1: 1K5, Resistor_SMD:R_0805_2012Metric, F.Cu at (121.6, 75.0)
- added R2: 1K, Resistor_SMD:R_0805_2012Metric, F.Cu at (134.3, 76.5)
- added R5: 68, Resistor_SMD:R_0805_2012Metric, F.Cu at (121.0, 93.2)
- added R7: 68, Resistor_SMD:R_0805_2012Metric, F.Cu at (126.5, 94.2)
- added U1: ATtiny85V-10S, Package_SO:SOIC-8W_5.3x5.3mm_P1.27mm, F.Cu at (128.0, 87.5)
Routing:
- net (no net): track 0.00 -> 355.6 mm
- net GND: track 0.00 -> 24.5 mm
- net /D+: track 0.00 -> 22.3 mm
Other:
- board outline added: 28.8 x 59.3 mm
