File: keyfob.kicad_sch (KiCad schematic)
At the start: 6 parts, among them U1 ATtiny85V-10S

Commit message: Initial commit
Other:
- moved on the sheet: C2
Changed lines of the file:
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@@
 	(paper "A4")
 	(junction
-		(at 142.24 113.03)
+		(at 142.24 102.87)
 		(diameter 0)
 		(color 0 0 0 0)
 	)
 	(junction
-		(at 142.24 120.65)
+		(at 142.24 110.49)
 		(diameter 0)
 		(color 0 0 0 0)
@@
 	(wire
 		(pts
-			(xy 129.54 113.03) (xy 142.24 113.03)
+			(xy 129.54 102.87) (xy 142.24 102.87)
 		)
 		(stroke
@@
 	(wire
 		(pts
-			(xy 142.24 107.95) (xy 142.24 113.03)
+			(xy 142.24 97.79) (xy 142.24 102.87)
 		)
 		(stroke
@@
 	(wire
 		(pts
-			(xy 129.54 120.65) (xy 142.24 120.65)
+			(xy 129.54 110.49) (xy 142.24 110.49)
 		)
 		(stroke
@@
 	(wire
 		(pts
-			(xy 142.24 120.65) (xy 142.24 124.46)
+			(xy 142.24 110.49) (xy 142.24 114.3)
 		)
 		(stroke
@@
 	(symbol
 		(lib_id "Device:C")
-		(at 129.54 116.84 0)
+		(at 129.54 106.68 0)
 		(unit 1)
 		(exclude_from_sim no)
@@
 		(dnp no)
 		(property "Reference" "C1"
-			(at 148.336 146.558 0)
+			(at 148.844 135.382 0)
 			(effects
 				(font
@@
 				)
 				(justify left)
+				(hide yes)
 			)
 		)
 		(property "Value" "4.7uf"
-			(at 133.35 118.1099 0)
+			(at 133.35 107.9499 0)
 			(effects
 				(font
@@
 		)
 		(property "Footprint" ""
-			(at 130.5052 120.65 0)
+			(at 130.5052 110.49 0)
 			(effects
 				(font
@@
 		)
 		(property "Datasheet" "~"
-			(at 129.54 116.84 0)
+			(at 129.54 106.68 0)
 			(effects
 				(font
@@
 		)
 		(property "Description" "Unpolarized capacitor"
-			(at 129.54 116.84 0)
+			(at 129.54 106.68 0)
 			(effects
 				(font
@@
 	(symbol
 		(lib_id "power:VCC")
-		(at 142.24 107.95 0)
+		(at 142.24 97.79 0)
 		(unit 1)
 		(exclude_from_sim no)
@@
 		(fields_autoplaced yes)
 		(property "Reference" "#PWR01"
-			(at 142.24 111.76 0)
+			(at 142.24 101.6 0)
 			(effects
 				(font
@@
 		)
 		(property "Value" "+5V"
-			(at 142.24 102.87 0)
-			(effects
-				(font
-					(size 1.27 1.27)
-				)
-			)
-		)
-		(property "Footprint" ""
-			(at 142.24 107.95 0)
+			(at 142.24 92.71 0)
+			(effects
+				(font
+					(size 1.27 1.27)
+				)
+			)
+		)
+		(property "Footprint" ""
+			(at 142.24 97.79 0)
 			(effects
 				(font
@@
 		)
 		(property "Datasheet" ""
-			(at 142.24 107.95 0)
+			(at 142.24 97.79 0)
 			(effects
 				(font
@@
 		)
 		(property "Description" "Power symbol creates a global label with name \"VCC\""
-			(at 142.24 107.95 0)
+			(at 142.24 97.79 0)
 			(effects
 				(font
@@
 	(symbol
 		(lib_id "power:GND")
-		(at 142.24 124.46 0)
+		(at 142.24 114.3 0)
 		(unit 1)
 		(exclude_from_sim no)
@@
 		(fields_autoplaced yes)
 		(property "Reference" "#PWR02"
-			(at 142.24 130.81 0)
+			(at 142.24 120.65 0)
 			(effects
 				(font
@@
 		)
 		(property "Value" "GND"
-			(at 142.24 129.54 0)
-			(effects
-				(font
-					(size 1.27 1.27)
-				)
-			)
-		)
-		(property "Footprint" ""
-			(at 142.24 124.46 0)
+			(at 142.24 119.38 0)
+			(effects
+				(font
+					(size 1.27 1.27)
+				)
+			)
+		)
+		(property "Footprint" ""
+			(at 142.24 114.3 0)
 			(effects
 				(font
@@
 		)
 		(property "Datasheet" ""
-			(at 142.24 124.46 0)
+			(at 142.24 114.3 0)
 			(effects
 				(font
@@
 		)
 		(property "Description" "Power symbol creates a global label with name \"GND\" , ground"
-			(at 142.24 124.46 0)
+			(at 142.24 114.3 0)
 			(effects
 				(font
@@
 	(symbol
 		(lib_id "Device:C")
-		(at 142.24 116.84 0)
+		(at 142.24 106.68 0)
 		(unit 1)
 		(exclude_from_sim no)
@@
 		(fields_autoplaced yes)
 		(property "Reference" "C2"
-			(at 146.05 115.5699 0)
+			(at 146.05 105.4099 0)
 			(effects
 				(font
@@
 		)
 		(property "Value" "0.1uf"
-			(at 146.05 118.1099 0)
+			(at 146.05 107.9499 0)
 			(effects
 				(font
@@
 		)
 		(property "Footprint" ""
-			(at 143.2052 120.65 0)
+			(at 143.2052 110.49 0)
 			(effects
 				(font
@@
 		)
 		(property "Datasheet" "~"
-			(at 142.24 116.84 0)
+			(at 142.24 106.68 0)
 			(effects
 				(font
@@
 		)
 		(property "Description" "Unpolarized capacitor"
-			(at 142.24 116.84 0)
-			(effects
-				(font
+			(at 142.24 106.68 0)
+			(effects
+				(font

Commit message: Updated the Schematic Design
Parts:
- added BT1: Battery_Cell, symbol Device:Battery_Cell
- added D2, D3: 3.6V, symbol Device:D_Zener
- added D4: D_Schottky, symbol Device:D_Schottky
- added J2: USB_A, symbol Connector:USB_A
- added PWR1: LED, symbol Device:LED
- added R1: 1K5, symbol Device:R
- added R2: 1K, symbol Device:R
- added R5, R7: 68, symbol Device:R
- added SW2: SW_SPDT_321, symbol Switch:SW_SPDT_321
- BZ1: value Buzzer -> BUZZER
Connections:
- net +5V: now also D4.2 (A), PWR1.1 (K), R1.1, SW2.1 (C)
- net GND: now also BT1.1 (+), D2.2 (A), D3.2 (A), J2.4 (GND), R2.1
- net VCC: now also SW2.2 (B); no longer BZ1.1 (+)
- net BUZZER: now reaches U1.1 (~{RESET}/PB5)
- net BUZZER: now also BZ1.1 (+)
- net PB4: now reaches U1.2 (XTAL1/PB3)
- net PB4: now also R7.1
- net PB3: now reaches U1.3 (XTAL2/PB4)
- net PB3: now also R5.2
- net BLUE: now reaches U1.5 (AREF/PB0)
- net BLUE: now also D1.2 (RA)
- net GREEN: now reaches U1.6 (PB1)
- net GREEN: now also D1.3 (GA)
- net RED: now reaches U1.7 (PB2)
- net RED: now also D1.4 (BA)
- new net: PWR1.2 (A), R2.2
- new net: D4.1 (K), J2.1 (VBUS)
- new net Cell Switch: BT1.2 (-), SW2.3 (A)
- new net D+: D3.1 (K), J2.3 (D+), R7.2
- new net D-: D2.1 (K), J2.2 (D-), R1.2, R5.1
- no-connect marks 0 -> 1
Other:
- note added: "USB A and Battery and Switch Connection"
- moved on the sheet: BZ1, C2, D1

Commit message: Upadated the Schematic and PCB Design
Parts:
- removed BT1: Battery_Cell, symbol Device:Battery_Cell
- removed SW2: SW_SPDT_321, symbol Switch:SW_SPDT_321
- BZ1: footprint (none) -> Buzzer_Beeper:Buzzer_15x7.5RM7.6
- C1, C2: footprint (none) -> Capacitor_SMD:C_Elec_3x5.4
- D1: footprint (none) -> LED_SMD:LED_RGB_1210
- D2, D3, D4: footprint (none) -> Diode_SMD:D_0805_2012Metric
- H1: footprint (none) -> MountingHole:MountingHole_4mm
- J2: footprint (none) -> Connector_USB:USB_A_Molex_67643_Horizontal
- PWR1: footprint (none) -> LED_SMD:LED_0805_2012Metric
- R1, R2, R5, R7: footprint (none) -> Resistor_SMD:R_0805_2012Metric
Other:
- moved on the sheet: C2, D2, D3, D4, J2, PWR1, R1, R2, R5, R7

Commit message: PCB layout done
Other:
- moved on the sheet: C2, D3, D4, J2, PWR1, R2, R7
